File: pcb/stat-monitor.sch (KiCad schematic (older format))
At the start: 1 part

Commit message: Added finalized PCB, initial firmware
Parts:
- added C1, C2: 33pF, Capacitor_SMD:C_0603_1608Metric_Pad1.08x0.95mm_HandSolder, symbol Device:C_Small
- added C3, C4: 1uF, Capacitor_SMD:C_0603_1608Metric_Pad1.08x0.95mm_HandSolder, symbol Device:C_Small
- added C5, C6: 0.1uF, Capacitor_SMD:C_0603_1608Metric_Pad1.08x0.95mm_HandSolder, symbol Device:C_Small
- added F1: 0.5A, Fuse:Fuse_1206_3216Metric_Pad1.42x1.75mm_HandSolder, symbol Device:Fuse_Polarized_Small
- added J1: Conn_01x04, Connector_PinSocket_2.54mm:PinSocket_1x04_P2.54mm_Vertical, symbol Connector_Generic:Conn_01x04
- added J2: Conn_01x07, Connector_PinHeader_2.54mm:PinHeader_1x07_P2.54mm_Vertical, symbol Connector_Generic:Conn_01x07
- added R1, R2: 22, Resistor_SMD:R_0603_1608Metric_Pad0.98x0.95mm_HandSolder, symbol Device:R_Small
- added R3, R4: 10k, Resistor_SMD:R_0603_1608Metric_Pad0.98x0.95mm_HandSolder, symbol Device:R_Small
- added SW1: SW_Push, Resistor_SMD:R_0805_2012Metric_Pad1.20x1.40mm_HandSolder, symbol Switch:SW_Push
- added Y1: 16M, parts:ECS-160-20-46X, symbol Device:Crystal_Small
- gave numbers to parts that had none: 1
Connections:
- net at U1.1 (XTAL1): now also C1.1, Y1.1
- net at U1.13 (~HWB~/PD7): now also R4.2
- net at U1.15 (PB1): now also J2.3 (Pin_3)
- net at U1.16 (PB2): now also J2.4 (Pin_4)
- net at U1.18 (PB4): now also J2.5 (Pin_5)
- net at U1.2 (PC0/XTAL2): now also C2.1, Y1.2
- net at U1.24 (PC1/~RESET): now also R3.1, SW1.2
- net at U1.27 (UCAP): now also C3.1
- net GND: now reaches U1.28 (UGND)
- net GND: now also U1.3 (GND), C1.2, C2.2, C3.2, C4.2, C5.2, C6.2, J1.4 (Pin_4), J2.1 (Pin_1), J2.6 (Pin_6), J2.7 (Pin_7), R4.1, SW1.1
- net D2+: now reaches U1.29 (D+)
- net D2+: now also R1.1
- net D2-: now reaches U1.30 (D-)
- net D2-: now also R2.1
- net +5V: now reaches U1.31 (UVCC)
- net +5V: now also U1.32 (AVCC), U1.4 (VCC), C4.1, C5.1, C6.1, F1.2, J2.2 (Pin_2), R3.2
- new net: F1.1, J1.1 (Pin_1)
- new net D1+: J1.3 (Pin_3), R1.2
- new net D1-: J1.2 (Pin_2), R2.2
